File: Rpi_esp_iot/_autosave-Rpi_esp_iot.kicad_sch (KiCad schematic)
At the start: 145 parts, among them J1 Conn_01x03, J2 U.FL-R-SMT-1(80), J3 USB_C_Receptacle_USB2.0_16P, J4 7111S2015X02LF, Q1 MMDT3904, SW1 SW_SPST, SW2 SW_SPST, U1 ST4SI2M0020TPIFW, U2 RASPBERRYPI-ZERO, U3 SHT30-DIS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

Commit message: Add eSIM connections and reorganize schematic layout
Parts:
- added R40, R41, R55, R56: 0R, Resistor_SMD:R_0402_1005Metric, symbol Device:R
- added TP24, TP25, TP26: TestPoint, PAD, symbol Connector:TestPoint
Connections:
- net ESIM_CLK: now also R40.1
- net ESIM_RST: now also R41.1
- net ESIM_VCC: now also R56.1
- net at R19.2, U5.30 (SIM_VDD): now also R56.2
- net at R18.2, U5.33 (SIM_RST): now also R55.2
- net ESIM_DATA: now reaches C41.2, R51.1, R52.2
- net ESIM_DATA: now also R55.1
- net at U5.24 (USB_VBUS): now also TP24.1
- net at U5.27 (USB_DP): now also TP26.1
- net at U5.28 (USB_DM): now also TP25.1
- net at R17.2, U5.31 (SIM_DATA): now also R41.2
- net at R16.2, U5.32 (SIM_CLK): now also R40.2
- no-connect marks 1 -> 5
Other:
- note added: "Level Sifter i2c smbus dedicated no usb connection on rpi and sim BQ24650 solar carger module Sourcing"
- note removed: "Level Sifter i2c smbus dedicated no usb connection on rpi and sim BQ24650 solar carger module Esim Connection Sourcing"
- note removed: "SOLAR INVERTER"
- moved on the sheet: C17, C18, C23, C24, C25, C26, C33, C34, C35, D5, FB1, J3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
