File: Rpi_esp_iot/Rpi_esp_iot.kicad_sch (KiCad schematic)
At the start: 145 parts, among them J1 Conn_01x03, J2 U.FL-R-SMT-1(80), J3 USB_C_Receptacle_USB2.0_16P, J4 7111S2015X02LF, Q1 MMDT3904, SW1 SW_SPST, SW2 SW_SPST, U1 ST4SI2M0020TPIFW, U2 RASPBERRYPI-ZERO, U3 SHT30-DIS, U4 MLX90614ESF-AAA-000-TU-ND, U5 SIM7070G, U6 ESP32-C6-MINI-1, U7 NXB0104PWJ, U9 MCP6001x-LT

Commit message: Level shifter is replaced to PCA9360 i2c bus dedicated
Parts:
- removed C42, C44: 100nF, Capacitor_SMD:C_0402_1005Metric, symbol Device:C_Small
- removed C43, C45: 1uF, Capacitor_SMD:C_0402_1005Metric, symbol Device:C_Small
- removed R53, R54: 10K, Resistor_SMD:R_0402_1005Metric, symbol Device:R_Small
- removed TP14, TP15, TP16, TP17: TestPoint, PAD, symbol Connector:TestPoint
- removed U7: NXB0104PWJ, NXB0104PWJ:SOP65P640X120-14N, symbol NXB0104PWJ:NXB0104PWJ
- added C46: 100pF, Capacitor_SMD:C_0402_1005Metric, symbol Device:C_Small
- added R40, R41, R55, R56: 0R, Resistor_SMD:R_0402_1005Metric, symbol Device:R
- added R57, R58: 10K, Resistor_SMD:R_0402_1005Metric, symbol Device:R_Small
- added R59: 200K, Resistor_SMD:R_0402_1005Metric, symbol Device:R_Small
- added TP24, TP25, TP26: TestPoint, PAD, symbol Connector:TestPoint
- added U8: PCA9306DCTR, PCA9306DCTR:SOP65P400X130-8N, symbol PCA9306DCTR:PCA9306DCTR
Connections:
- net +5V_SEN is gone; now on net +5V_RPi: R13.1, R14.1
- net +3V3_RPI: now also R57.1, R58.1, U8.2 (VREF1)
- net +5V_RPi: now also C46.2, R59.1, U8.7 (VREF2)
- net ESIM_CLK: now also R40.1
- net ESIM_RST: now also R41.1
- net ESIM_VCC: now also R56.1
- net GND: now also C46.1, U8.1 (GND)
- net RPI_SCL: now also R57.2, U8.3 (SCL1); no longer R14.2, U3.4 (SCL), U4.1 (SCL/VZ)
- net RPI_SDA: now also R58.2, U8.4 (SDA1); no longer R13.2, U3.1 (SDA), U4.2 (SDA/PWM)
- net at R19.2, U5.30 (SIM_VDD): now also R56.2
- net at R18.2, U5.33 (SIM_RST): now also R55.2
- net ESIM_DATA: now reaches C41.2, R51.1, R52.2
- net ESIM_DATA: now also R55.1
- net at U5.24 (USB_VBUS): now also TP24.1
- net at U5.27 (USB_DP): now also TP26.1
- net at U5.28 (USB_DM): now also TP25.1
- net at R17.2, U5.31 (SIM_DATA): now also R41.2
- net at R16.2, U5.32 (SIM_CLK): now also R40.2
- new net: R59.2, U8.8 (EN)
- new net SNS_I2C_SCL: R14.2, U3.4 (SCL), U4.1 (SCL/VZ), U8.6 (SCL2)
- new net SNS_I2C_SDA: R13.2, U3.1 (SDA), U4.2 (SDA/PWM), U8.5 (SDA2)
- no-connect marks 1 -> 5
Other:
- note added: "Level Sifter i2c smbus dedicated no usb connection on rpi and sim BQ24650 solar carger module Sourcing"
- note removed: "Level Sifter i2c smbus dedicated no usb connection on rpi and sim BQ24650 solar carger module Esim Connection Sourcing"
- note removed: "SOLAR INVERTER"
- moved on the sheet: AE1, C1, C10, C17, C18, C19, C2, C20, C23, C24, C25, C26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

Commit message: Solar Charge Controller added and layout is improved
Parts:
- removed TP18: TestPoint, PAD, symbol Connector:TestPoint
- added C42: 2.2uF, Capacitor_SMD:C_1210_3225Metric_Pad1.33x2.70mm_HandSolder, symbol Device:C_Small
- added C43, C44, C53: 1uF, Capacitor_SMD:C_0805_2012Metric_Pad1.18x1.45mm_HandSolder, symbol Device:C_Small
- added C45, C51: 0.1uF, Capacitor_SMD:C_0402_1005Metric, symbol Device:C_Small
- added C48, C49: 10uF, Capacitor_SMD:C_1210_3225Metric_Pad1.33x2.70mm_HandSolder, symbol Device:C_Small
- added C50: 4.7uF, Capacitor_SMD:C_1210_3225Metric_Pad1.33x2.70mm_HandSolder, symbol Device:C_Small
- added C52: 22pF, Capacitor_SMD:C_0603_1608Metric_Pad1.08x0.95mm_HandSolder, symbol Device:C_Small
- added D3: PDS1040, Diode_SMD:D_SMB, symbol Diode:S2JTR
- added D4, D8: LTST-C190GKT, symbol Device:LED
- added D9: BAT54C, Diode_SMD:D_SMC, symbol Diode:B320
- added J5: Barrel_Jack_MountingPin, symbol Connector:Barrel_Jack_MountingPin
- added L1: 10uH, symbol Device:L
- added Q2, Q5: NMOS, symbol Simulation_SPICE:NMOS
- added Q3, Q4: Si7288, symbol Simulation_SPICE:NMOS
- added R53: 10R, Resistor_SMD:R_1206_3216Metric_Pad1.30x1.75mm_HandSolder, symbol Device:R_Small
- added R54: 2R, symbol Device:R_Small
- added R60, R69: 5.23K, Resistor_SMD:R_0402_1005Metric, symbol Device:R_Small
- added R61: 30.1K, Resistor_SMD:R_0402_1005Metric, symbol Device:R_Small
- added R62, R67: 499K, Resistor_SMD:R_0402_1005Metric, symbol Device:R_Small
- added R63: 36K, Resistor_SMD:R_0402_1005Metric, symbol Device:R_Small
- added R64, R65, R70, R71: 10K, Resistor_SMD:R_0402_1005Metric, symbol Device:R_Small
- added R66: 20mR, Resistor_SMD:R_0402_1005Metric, symbol Device:R_Small
- added R68: 100K, Resistor_SMD:R_0402_1005Metric, symbol Device:R_Small
- added TH1: Thermistor_NTC, symbol Device:Thermistor_NTC
- added U7: BQ24650RVAT, BQ24650RVAT:QFN50P350X350X100-17N, symbol BQ24650RVAT:BQ24650RVAT
- U1: Manufacturer (none) -> STMicroelectronics; Manufacturer Part Number (none) -> ST4SI2M0020TPIFW
- U2: Manufacturer (none) -> Raspberry Pi; Manufacturer Part Number (none) -> RASPBERRYPI-ZERO
- U4: Manufacturer (none) -> Melexis; Manufacturer Part Number (none) -> MLX90614ESF-AAA-000-TU
- U5: Manufacturer (none) -> simcom wireless solutions limited; Manufacturer Part Number (none) -> SIM7070G
- U8: Manufacturer (none) -> Texas Instruments; Manufacturer Part Number (none) -> PCA9306DCTR
- VR1, VR2, VR3: Manufacturer (none) -> Texas Instruments; Manufacturer Part Number (none) -> TPSM863252RDXR
Connections:
- net +Vsys is gone; now on net +Vbat: C3.1, C4.1, C7.1, C8.1, R4.1, R8.1, VR2.1 (VIN), VR3.1 (VIN)
- net +3V3_RPI: now also Q5.2 (G), R70.1
- net +5V_RPi: now also R71.1
- net +Vbat: now also C49.2, C50.1, C51.2, C52.1, R66.2, R67.2, R69.1, U7.9 (SRN)
- net BATTERY: now also U6.24 (IO18)
- net GND: now also C42.1, C43.1, C44.1, C48.1, C49.1, C50.2, C53.2, J5.2, Q2.3 (S), Q4.3 (S), R61.2, R63.2, R68.1, TH1.2, U7.11 (GND)
- net SHT_ALT: now also Q5.1 (D), R71.2
- net SIM_VCC: now also D1.2 (A), D2.2 (A)
- net VBAT: no longer D1.2 (A), D2.2 (A)
- net SHT_ALT_Rpi: now reaches U2.29 (GPIO5)
- net SHT_ALT_Rpi: now also Q5.3 (S), R70.2
- new net: D4.1 (K), U7.5 (STAT2)
- new net: D4.2 (A), R64.2
- new net: C43.2, R53.2, U7.1 (VCC)
- new net: C51.1, L1.2, R66.1, U7.10 (SRP)
- new net: C44.2, D9.2 (A), U7.12 (REGN)
- new net: Q4.2 (G), U7.13 (LODRV)
- new net: C45.2, L1.1, Q3.3 (S), Q4.1 (D), U7.14 (PH)
- new net: Q3.2 (G), U7.15 (HIDRV)
- new net: C45.1, D9.1 (K), U7.16 (BTST)
- new net: Q2.1 (D), R62.2, R63.1, U7.2 (MPPSET)
- new net: D8.1 (K), U7.3 (STAT1)
- new net: C53.1, R60.1, U7.6 (VREF)
- new net: C52.2, R67.1, R68.2, U7.8 (VFB)
- new net: C48.2, D3.1 (K), Q3.1 (D), R53.1
- new net: D8.2 (A), R65.2
- new net: C42.2, R54.2
- new net BAT_TEMP: R60.2, R61.1, R69.2, TH1.1, U7.4 (TS)
- new net VIN: D3.2 (A), J5.1, Q2.2 (G), R54.1, R62.1, R64.1, R65.1
Other:
- note added: "Battery Pack"
- note added: "Battery full"
- note added: "Charging"
- note added: "SOLAR CHARGE CONTROLLER"
- note added: "Solar cell"
- note added: "Sourcing"
- note added: "Thermister"
- note removed: "I2C PULL UPS"
- note removed: "Level Sifter i2c smbus dedicated no usb connection on rpi and sim BQ24650 solar carger module Sourcing"
- moved on the sheet: AE1, C11, C12, C13, C14, C15, C16, C17, C18, C19, C20, C21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

Commit message: Sourcing Complete + Added all Components to PCB + Resolved errors
Parts:
- AE1: now not fitted
- C1, C5, C9: Manufacturer (none) -> muRata; Manufacturer Part Number (none) -> GRM1555C1H220JA01D; Supplier (none) -> LCSC; Supplier Part Number (none) -> C76960
- C10, C2, C6: Manufacturer (none) -> Samsung Electro-Mechanics; Manufacturer Part Number (none) -> CL05C330JB5NNNC; Supplier Part Number (none) -> C70465
- C11, C12, C13, C14, C17, C19, C21, C23, C25, C27, C28, C31, C32, C36, C37, C41: Manufacturer (none) -> YAGEO; Manufacturer Part Number (none) -> CC0402KRX7R7BB104; Supplier Part Number (none) -> C60474
- C15, C24, C26, C33, C34, C35: Manufacturer (none) -> Samsung Electro-Mechanics; Manufacturer Part Number (none) -> CL05A105KP5NNNC; Supplier Part Number (none) -> C14445
- C16: value 470Uf -> 470uf; footprint Resistor_SMD:R_0402_1005Metric -> Capacitor_Tantalum_SMD:CP_EIA-7343-15_Kemet-W_HandSolder; Manufacturer (none) -> Kyocera AVX; Manufacturer Part Number (none) -> TAJD477K006RNJ; Supplier Part Number (none) -> C7229
- C18, C20: Manufacturer (none) -> Samsung Electro-Mechanics; Manufacturer Part Number (none) -> CL05A475MP5NRNC; Supplier Part Number (none) -> C23733
- C22, C38, C39, C40: Manufacturer (none) -> Samsung Electro-Mechanics; Manufacturer Part Number (none) -> CL05A226MQ5QUNC; Supplier Part Number (none) -> C105226
- C29, C3, C7: Manufacturer (none) -> Samsung Electro-Mechanics; Manufacturer Part Number (none) -> CL05A106MP5NUNC; Supplier Part Number (none) -> C315248
- C30, C4, C45, C51, C8: value 0.1uF -> 100nF; Manufacturer (none) -> YAGEO; Manufacturer Part Number (none) -> CC0402KRX7R7BB104; Supplier Part Number (none) -> C60474
- C42: Manufacturer (none) -> KEMET; Manufacturer Part Number (none) -> C1210C225K1RACAUTO; Supplier Part Number (none) -> C561798
- C43, C44, C53: Manufacturer (none) -> KEMET; Manufacturer Part Number (none) -> C0805C105K5RACAUTO; Supplier Part Number (none) -> C3874210
- C46: value 100pF -> 1000pF; Manufacturer (none) -> muRata; Manufacturer Part Number (none) -> GRM1555C1H102JA01D; Supplier Part Number (none) -> C76947
- C48, C49: Manufacturer (none) -> YAGEO; Manufacturer Part Number (none) -> CC1210KKX7R9BB106; Supplier Part Number (none) -> C596319
- C50: Manufacturer (none) -> Samsung Electro-Mechanics; Manufacturer Part Number (none) -> CL32B475KBUYNNE; Supplier Part Number (none) -> C170099
- C52: Manufacturer (none) -> KEMET; Manufacturer Part Number (none) -> C0603C220K5RACAUTO; Supplier Part Number (none) -> C2169931
- D1: footprint (none) -> LED_SMD:LED_0402_1005Metric_Pad0.77x0.64mm_HandSolder; Manufacturer (none) -> XINGLIGHT; Manufacturer Part Number (none) -> XL-1005SURC; Supplier Part Number (none) -> C25503345
- D2: footprint (none) -> LED_SMD:LED_0402_1005Metric_Pad0.77x0.64mm_HandSolder; Manufacturer (none) -> XINGLIGHT; Manufacturer Part Number (none) -> XL-1005UGC; Supplier Part Number (none) -> C965793
- D3: footprint Diode_SMD:D_SMB -> Diode_SMD:D_PowerDI-5; Manufacturer (none) -> DIODES; Manufacturer Part Number (none) -> PDS1040-13; Supplier Part Number (none) -> C110512
- D4, D8: footprint (none) -> LED_SMD:LED_0603_1608Metric_Pad1.05x0.95mm_HandSolder; Manufacturer (none) -> LITEON; Manufacturer Part Number (none) -> LTST-C190GKT; Supplier Part Number (none) -> C125093
- D5: value S2JTR -> SS54; footprint Diode_SMD:D_SMB -> Diode_SMD:D_SMA_Handsoldering; Manufacturer (none) -> MDD(Microdiode Semiconductor); Manufacturer Part Number (none) -> SS54; Supplier Part Number (none) -> C22452
- D6, D7: footprint Package_TO_SOT_SMD:SOT-23-6 -> Package_TO_SOT_SMD:SOT-23-6_Handsoldering; Manufacturer (none) -> ST; Manufacturer Part Number (none) -> ESDA6V1BC6; Supplier Part Number (none) -> C495220
- D9: footprint Diode_SMD:D_SMC -> Package_TO_SOT_SMD:SOT-23-3; Manufacturer (none) -> JSMSEMI; Manufacturer Part Number (none) -> BAT54C; Supplier Part Number (none) -> C916424
- FB1: Manufacturer (none) -> TDK; Manufacturer Part Number (none) -> MPZ2012S601AT000; Supplier Part Number (none) -> C21519
- J1: footprint U.FL-R-SMT-1(80) -> Connector_Coaxial:U.FL_Hirose_U.FL-R-SMT-1_Vertical; Manufacturer (none) -> HRS; Manufacturer Part Number (none) -> U.FL-R-SMT-1(80); Supplier Part Number (none) -> C88374
- J2: value U.FL-R-SMT-1(80) -> Conn_01x03; footprint (none) -> Connector_Coaxial:U.FL_Hirose_U.FL-R-SMT-1_Vertical; Manufacturer (none) -> HRS; Manufacturer Part Number (none) -> U.FL-R-SMT-1(80); Supplier Part Number (none) -> C88374
- J3: footprint Connector_USB:USB_C_Receptacle_HRO_TYPE-C-31-M-12 -> Connector_USB:USB_C_Receptacle_GCT_USB4115-03-C; Manufacturer (none) -> Global Connector Technology; Manufacturer Part Number (none) -> USB4115-03-C; Supplier Part Number (none) -> C5250720
- J4: footprint (none) -> 7111S2015X02LF:FCI_7111S2015X02LF; Manufacturer (none) -> Amphenol; Manufacturer Part Number (none) -> 7111S2015X02LF; Supplier Part Number (none) -> C598923
- J5: footprint (none) -> Connector_BarrelJack:BarrelJack_GCT_DCJ200-10-A_Horizontal
- L1: footprint (none) -> Inductor_SMD:L_Vishay_IHLP-2525; Manufacturer (none) -> VISHAY; Manufacturer Part Number IHLP-2525CZ -> IHLP2525CZER100M01; Supplier Part Number (none) -> C540965
- Q1: Manufacturer (none) -> TWGMC; Manufacturer Part Number (none) -> MMDT3904; Supplier Part Number (none) -> C5204740
- Q2, Q5: footprint (none) -> Package_TO_SOT_SMD:SOT-23_Handsoldering; Manufacturer (none) -> VISHAY; Manufacturer Part Number (none) -> 2N7002K-T1-GE3; Supplier Part Number (none) -> C81445
- Q3, Q4: footprint (none) -> Package_SO:PowerPAK_SO-8_Dual; Manufacturer (none) -> VISHAY; Manufacturer Part Number (none) -> SI7288DP-T1-GE3; Supplier Part Number (none) -> C126988
- R1, R10, R12, R13, R14, R15, R32, R36, R37, R42, R43, R57, R58, R6, R64, R65, R70, R71: Manufacturer (none) -> YAGEO; Manufacturer Part Number (none) -> RC0402FR-0710KL; Supplier Part Number (none) -> C60490
- R11, R3, R7: Manufacturer (none) -> YAGEO; Manufacturer Part Number (none) -> RC0402FR-0730KL; Supplier Part Number (none) -> C138008
- R16, R17, R18, R19, R20, R21, R22, R23, R31, R34, R38, R39, R40, R41, R44, R45, R46, R47, R48, R49, R50, R51, R52, R55, R56: Manufacturer (none) -> YAGEO; Manufacturer Part Number (none) -> RC0402FR-070RL; Supplier Part Number (none) -> C106231
- R2: footprint Resistor_SMD:R_0402_1005Metric -> Resistor_SMD:R_0603_1608Metric_Pad0.98x0.95mm_HandSolder; Manufacturer (none) -> Viking; Manufacturer Part Number (none) -> ARG03BTC1353N; Supplier Part Number (none) -> C1509632
- R24: Manufacturer (none) -> YAGEO; Manufacturer Part Number (none) -> RC0402FR-07330RL; Supplier Part Number (none) -> C105875
- R25, R4, R8: Manufacturer (none) -> YAGEO; Manufacturer Part Number (none) -> RT0402BRD0748K7L; Supplier Part Number (none) -> C852805
- R26: Manufacturer (none) -> YAGEO; Manufacturer Part Number (none) -> RC0402FR-07120RL; Supplier Part Number (none) -> C114758
- R27, R29: Manufacturer (none) -> YAGEO; Manufacturer Part Number (none) -> RC0402FR-074K7L; Supplier Part Number (none) -> C105871
- R28, R30: Manufacturer (none) -> YAGEO; Manufacturer Part Number (none) -> RC0402FR-0747KL; Supplier Part Number (none) -> C93943
- R33, R35: Manufacturer (none) -> YAGEO; Manufacturer Part Number (none) -> RC0402FR-0724KL; Supplier Part Number (none) -> C138026
- R5: Manufacturer (none) -> YAGEO; Manufacturer Part Number (none) -> RC0402FR-07220KL; Supplier Part Number (none) -> C138030
- R53: Manufacturer (none) -> YAGEO; Manufacturer Part Number (none) -> RC1206FR-0710RL; Supplier Part Number (none) -> C108080
- R54: footprint (none) -> Resistor_SMD:R_2512_6332Metric_Pad1.40x3.35mm_HandSolder; Manufacturer (none) -> RESI; Manufacturer Part Number (none) -> MFCR2512F2R00Q9R; Supplier Part Number (none) -> C42415569
- R59: Manufacturer (none) -> FOJAN; Manufacturer Part Number (none) -> FRC0402F2003TS; Supplier Part Number (none) -> C2906866
- R60, R69: Manufacturer (none) -> Viking; Manufacturer Part Number (none) -> ARG02BTC5231; Supplier Part Number (none) -> C2684530
- R61: Manufacturer (none) -> UNI-ROYAL; Manufacturer Part Number (none) -> 0402WGF3012TCE; Supplier Part Number (none) -> C29402
- R62, R67: Manufacturer (none) -> YAGEO; Manufacturer Part Number (none) -> RC0402FR-07499KL; Supplier Part Number (none) -> C137971
- R63: Manufacturer (none) -> FOJAN; Manufacturer Part Number (none) -> FRC0402F3602TS; Supplier Part Number (none) -> C2930004
- R66: Manufacturer (none) -> JIERR; Manufacturer Part Number WSL1206R0200DEA -> JER1206F1R020; Supplier Part Number (none) -> C46634440
- R68: Manufacturer (none) -> YAGEO; Manufacturer Part Number (none) -> RC0402FR-07100KL; Supplier Part Number (none) -> C60491
- R9: Manufacturer (none) -> ChipNobo; Manufacturer Part Number (none) -> RK73H1ET1653F-CN; Supplier Part Number (none) -> C42396631
- SW1, SW2: footprint (none) -> Button_Switch_SMD:SW_SPST_SKQG_WithStem; Manufacturer C&K -> G-Switch; Manufacturer Part Number KMR231G LFS -> GT-TZ084B-H015-L1; Supplier DigiKey -> (none); Supplier Part Number 108-KMR231GLFSCT-ND -> C29780122
- TH1: footprint (none) -> Resistor_SMD:R_0402_1005Metric_Pad0.72x0.64mm_HandSolder; Manufacturer (none) -> cjiang; Manufacturer Part Number (none) -> FNTC0402X103F3380FB; Supplier Part Number (none) -> C41417281
- TP1, TP10, TP11, TP12, TP13, TP19, TP2, TP20, TP21, TP22, TP23, TP24, TP25, TP26, TP3, TP4, TP5, TP6, TP7, TP8, TP9: footprint PAD -> TestPoint:TestPoint_Pad_2.0x2.0mm
- U1: Supplier Part Number (none) -> C5267509
- U5: Supplier Part Number (none) -> C2892847
- U6: Manufacturer (none) -> ESPRESSIF; Manufacturer Part Number (none) -> ESP32-C6-MINI-1-N4; Supplier Part Number (none) -> C5736265
- U7: Supplier Part Number (none) -> C2876745
- U8: Supplier Part Number (none) -> C123752
- VR1, VR2, VR3: Supplier Part Number (none) -> C19632640
Connections:
- net +5V_RPi: no longer C46.2, R13.1, R14.1, U8.7 (VREF2)
- net DATA_EN: now also J4.7 (I/O); no longer J4.6 (I/O)
- net GND: now also J4.5 (GND); no longer J1.3 (Pin_3), J2.3 (Pin_3), J4.4 (GND)
- net at R59.2, U8.8 (EN): now also C46.2, R13.1, R14.1, U8.7 (VREF2)
Other:
- note removed: "Sourcing"
- moved on the sheet: R59

Commit message: Placement by usama
Parts:
- removed J4: 7111S2015X02LF, 7111S2015X02LF:FCI_7111S2015X02LF, symbol Connector:SIM_Card
- removed R52: 0R, Resistor_SMD:R_0402_1005Metric, symbol Device:R_Small
- added H1, H2, H3, H4, H5: MountingHole_Pad, MountingHole:MountingHole_3.2mm_M3_DIN965_Pad, symbol Mechanical:MountingHole_Pad
- added J6: SIM8066-6-1-14-01-A_REVA, Rpi_esp_iot:GCT_SIM8066-6-1-14-01-A_REVA, symbol Rpi_esp_iot:SIM8066-6-1-14-01-A_REVA
- R16, R17, R18, R19, TP19, TP20, TP21, TP22, TP23, TP5, TP6: now not fitted
- R42, R43: value 10K -> 5.1K
- TP1, TP10, TP11, TP12, TP13, TP2, TP24, TP25, TP26, TP3, TP4, TP7, TP8, TP9: now not fitted; now left out of the parts list
Connections:
- net CLK_EN: now also J6.C3 (CLK)
- net DATA_EN: now also J6.C7 (I/O)
- net ESIM_DATA: no longer C41.2
- net ESIM_VCC: now also C41.2, D7.4 (TVS3)
- net ES_DATA_EN: now also D7.6 (TVS4); no longer D7.4 (TVS3)
- net GND: now also H1.1, H2.1, H3.1, H4.1, H5.1, J6.C5 (GND), J6.G1 (GND), J6.G2 (GND), J6.G3 (GND), J6.G4 (GND)
- net RST_EN: now also J6.C2 (RST)
- net SIM_VCC: now also J6.C1 (VCC); no longer R19.1
- new net PSIM_VCC: R19.1
Other:
- moved on the sheet: C43, C44, C45

Commit message: Complete Placement + Partial modification in Schematic(Sim+simreset+Power Connection wit diode
Parts:
- removed J5: Barrel_Jack_MountingPin, Connector_BarrelJack:BarrelJack_GCT_DCJ200-10-A_Horizontal, symbol Connector:Barrel_Jack_MountingPin
- removed Q3, Q4: Si7288, Package_SO:PowerPAK_SO-8_Dual, symbol Simulation_SPICE:NMOS
- added D10: SS26, Diode_SMD:D_SMA_Handsoldering, symbol Diode:S2JTR
- added Q3, Q4: CSD18540Q5B, CSD18540Q5B:CSD18540Q5B, symbol 2026-04-24_21-06-56:CSD18540Q5B
- added Q6: MMDT3904, Package_TO_SOT_SMD:SOT-363_SC-70-6, symbol Transistor_BJT:MMDT3904
- added R52: 20k, Resistor_SMD:R_0402_1005Metric, symbol Device:R_Small
- added R72: 4.7K, Resistor_SMD:R_0402_1005Metric, symbol Device:R
- added R74: 47K, Resistor_SMD:R_0402_1005Metric, symbol Device:R
- added TP14, TP15: TestPoint, TestPoint:TestPoint_Pad_2.0x2.0mm, symbol Connector:TestPoint
- added TP16: BAT +, TestPoint:TestPoint_Pad_2.0x2.0mm, symbol Connector:TestPoint
- added TP17: BAT-, TestPoint:TestPoint_Pad_2.0x2.0mm, symbol Connector:TestPoint
- D5: value SS54 -> SS26; Manufacturer MDD(Microdiode Semiconductor) -> ElecSuper; Manufacturer Part Number SS54 -> SS26; Supplier (none) -> LCSC; Supplier Part Number C22452 -> C5350986
- J3: footprint Connector_USB:USB_C_Receptacle_GCT_USB4115-03-C -> USB4115_03_C:USB4115-03-C_GCT
Connections:
- net VBAT is gone; now on net SIM_VCC: U5.56 (VBAT), U5.57 (VBAT)
- net +5V_RPi: now also D10.1 (K)
- net +V_SUPPLY: now also D10.2 (A)
- net +Vbat: now also TP16.1
- net ESIM_VCC: now also R52.1
- net ES_DATA_EN: now also R52.2
- net GND: now also U2.14 (GND[4]), U7.17 (EPAD), Q4.3, TP15.1, TP17.1
- net SIM_PWRKEY: now also Q6.3 (C2); no longer U2.11 (GPIO17/GEN0)
- net VIN: now also TP14.1
- net at U7.13 (LODRV): now also Q4.2
- net at C45.2, L1.1, U7.14 (PH): now also Q3.3, Q4.1
- net at U7.15 (HIDRV): now also Q3.2
- net at C53.1, R60.1, U7.6 (VREF): now also U7.7 (TERM_EN)
- net at C48.2, D3.1 (K), R53.1: now also Q3.1
- new net: Q6.5 (B2), R72.2, R74.1
- new net: Q6.4 (E2), R74.2
- new net SIM_PWRKEY_Rpi: R72.1, U2.11 (GPIO17/GEN0)
Other:
- note added: "LEVEL SHIFT GPIO"
- note added: "SIM MODULE RESET / PWR KEY"
- moved on the sheet: C41, C42, C43, C44, C45, C48, C49, C50, C51, C52, C53, D3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

Commit message: Routing Complete
Parts:
- removed D10: SS26, Diode_SMD:D_SMA_Handsoldering, symbol Diode:S2JTR
- removed R46, R47, R48, R49, R50, R51: 0R, Resistor_SMD:R_0402_1005Metric, symbol Device:R_Small
- C45, C51: footprint Capacitor_SMD:C_0402_1005Metric -> Resistor_SMD:R_0805_2012Metric; Manufacturer Part Number CC0402KRX7R7BB104 -> CC0805KRX7R9BB104; Package (none) -> 0805; Supplier Part Number C60474 -> C49678
- R66: footprint Resistor_SMD:R_0402_1005Metric -> Resistor_SMD:R_1206_3216Metric_Pad1.30x1.75mm_HandSolder; Package (none) -> 1206
Connections:
- net +3.3V is gone; now on net +3.3V_ESP: R37.2
- net +3V3 is gone; now on net +3.3V_ESP: U9.5 (V+)
- net +V_SUPPLY is gone; now on net +Vbat: C29.1, C30.1, D5.1 (K), R25.1, VR1.1 (VIN)
- net CLK_EN is gone; now on net SIM_CLK: C39.1, D6.3 (TVS2), J6.C3 (CLK)
- net DATA_EN is gone; now on net SIM_DATA: C40.1, D6.6 (TVS4), J6.C7 (I/O)
- net ES_CLK_EN is gone; now on net ESIM_CLK: D7.3 (TVS2), U1.6 (CLK)
- net ES_DATA_EN is gone; now on net ESIM_DATA: D7.6 (TVS4), R52.2, U1.3 (I/O)
- net ES_RST_EN is gone; now on net ESIM_RST: D7.1 (TVS1), U1.7 (~{RESET})
- net PSIM_VCC is gone; now on net SIM_VCC: R19.1
- net RST_EN is gone; now on net SIM_RST: C38.1, D6.1 (TVS1), J6.C2 (RST)
- net GND: no longer R1.1, R25.2, VR1.6 (EN)
- net ESP_GPIO12_USB_D- renamed ESP_USB_D_N
- net ESP_GPIO13_USB_D+ renamed ESP_USB_D_P
- new net: R1.1, R25.2, VR1.6 (EN)
Other:
- moved on the sheet: C51
